File: Electrical/TestPlatformBoard1.1/LMC6482.sch (KiCad schematic (older format))
At the start: 7 parts, among them U3 LMC6482

Commit message: v1.0
Parts:
- R10, R11: value 5M -> 1M
Connections:
- net labels added: A+, B+
- net labels removed: A-, B-
Other:
- note removed: "ITS FUCKED, V- and A-/B- need to be switched\n"
Changed lines of the file:
@@
 	4950 3800 4750 3800
 Text HLabel 4550 2450 0    50   Input ~ 0
-A-
+A+
 Wire Wire Line
 	4950 2650 4700 2650
 Text HLabel 4550 3800 0    50   Input ~ 0
-B-
+B+
 $Comp
 L Device:R R10
@@
 P 5050 2100
 F 0 "R10" V 4843 2100 50  0000 C CNN
-F 1 "5M" V 4934 2100 50  0000 C CNN
+F 1 "1M" V 4934 2100 50  0000 C CNN
 F 2 "Resistors_SMD:R_1206_HandSoldering" V 4980 2100 50  0001 C CNN
 F 3 "~" H 5050 2100 50  0001 C CNN
@@
 P 5050 3450
 F 0 "R11" V 4843 3450 50  0000 C CNN
-F 1 "5M" V 4934 3450 50  0000 C CNN
+F 1 "1M" V 4934 3450 50  0000 C CNN
 F 2 "Resistors_SMD:R_1206_HandSoldering" V 4980 3450 50  0001 C CNN
 F 3 "~" H 5050 3450 50  0001 C CNN
@@
 Text HLabel 4600 4300 0    50   Input ~ 0
 V-
-Text Notes 6150 2950 0    50   ~ 0
-ITS FUCKED, V- and A-/B- need to be switched\n
 Wire Wire Line
 	4950 4000 4700 4000
