File: Electrical/TestPlatformBoard1.1/TestPlatformBoard.kicad_pcb (KiCad board)
At the start: 2 copper layers, 88.9 x 76.2 mm, 61 parts, among them IC1 CL520N3-G, IC2 CL520N3-G, IC3 TCR2EF33,LM(CT, IC4 ADC122S021CIMM_NOPB, IC5 DS2482-100, J1 Conn_01x04, J2 Conn_01x02_Male, J3 Conn_01x03_Male, J4 Conn_01x02_Male, J5 Conn_01x08_Male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

Commit message: v1.0
Parts:
- removed REF** (x4): MountingHole_3.7mm, Mounting_Holes:MountingHole_3.7mm
- removed REF** (x4): MountingHole_3.2mm_M3, Mounting_Holes:MountingHole_3.2mm_M3
- added J8: Conn_01x01_Male, Connectors_Samtec:SL-101-X-XX_1x01, F.Cu at (45.7, 53.0)
- added MH1: MountingHole, Mounting_Holes:MountingHole_3.2mm_M3, F.Cu at (10.3, 10.3)
- added MH2: MountingHole, Mounting_Holes:MountingHole_3.2mm_M3, F.Cu at (37.4, 10.3)
- added MH3: MountingHole, Mounting_Holes:MountingHole_3.2mm_M3, F.Cu at (37.4, 27.4)
- added MH4: MountingHole, Mounting_Holes:MountingHole_3.2mm_M3, F.Cu at (10.3, 27.4)
- added MH5: MountingHole, Mounting_Holes:MountingHole_3.7mm, F.Cu at (5.08, 5.08)
- added MH6: MountingHole, Mounting_Holes:MountingHole_3.7mm, F.Cu at (83.8, 5.08)
- added MH7: MountingHole, Mounting_Holes:MountingHole_3.7mm, F.Cu at (83.8, 71.1)
- added MH8: MountingHole, Mounting_Holes:MountingHole_3.7mm, F.Cu at (5.08, 71.1)
- added Q3: DMN3404, TO_SOT_Packages_SMD:SOT-23_Handsoldering, F.Cu at (38.0, 3.49)
- added Q7: AOD4184A, TO_SOT_Packages_SMD:TO-252-2, F.Cu at (45.4, 4.31)
- added R14: 33k, Resistors_SMD:R_0805_HandSoldering, F.Cu at (31.9, 4.16)
- added R15: 1k, Resistors_SMD:R_0805_HandSoldering, F.Cu at (34.9, 3.79)
- R10, R11: value 5M -> 1M
- R3: value 330 -> 1k
- moved D6 2.58 mm to (15.3, 72.9), turned to 180 degrees
- moved D3 2.56 mm to (30.7, 72.9), turned to 180 degrees
- moved D7 2.54 mm to (22.9, 72.9), turned to 180 degrees
- moved R3 0.22 mm to (75.1, 32.2), turned to 180 degrees
Connections:
- C10 pad 2: GNDA -> /LMC6482/B+
- C9 pad 2: GNDA -> /LMC6482/A+
- D4 pad 1: /LMC6482/B- -> /LMC6482/B+
- D5 pad 1: /LMC6482/A- -> /LMC6482/A+
- Q2 pad 3: Net-(D3-Pad2) -> Net-(D3-Pad1)
- Q4 pad 3: Net-(D6-Pad2) -> Net-(D6-Pad1)
- Q6 pad 3: Net-(D7-Pad2) -> Net-(D7-Pad1)
- R10 pad 2: GNDA -> /LMC6482/A+
- R11 pad 2: GNDA -> /LMC6482/B+
- R3 pad 1: Net-(Q3-Pad1) -> CTRL_Heater
- R3 pad 2: CTRL_Heater -> Net-(Q3-Pad1)
- R5 pad 1: Net-(D3-Pad1) -> Net-(D3-Pad2)
- R7 pad 1: Net-(D6-Pad1) -> Net-(D6-Pad2)
- R9 pad 1: Net-(D7-Pad1) -> Net-(D7-Pad2)
- U3 pad 2: /LMC6482/A- -> GNDA
- U3 pad 3: GNDA -> /LMC6482/A+
- U3 pad 5: GNDA -> /LMC6482/B+
- U3 pad 6: /LMC6482/B- -> GNDA
Routing:
- net GNDA: track 192.8 -> 86.9 mm, vias 17 -> 15
- net /LMC6482/A+: track 0.00 -> 56.3 mm
- net /LMC6482/A-: track 47.7 -> 0.00 mm
- net /LMC6482/B+: track 0.00 -> 33.2 mm
- net /LMC6482/B-: track 31.0 -> 0.00 mm
- net Net-(Q3-Pad1): track 32.2 -> 54.3 mm, vias 0 -> 2
- net +3V3: track 154.3 -> 175.2 mm
- net I2C_SCL: track 52.3 -> 71.2 mm, vias 0 -> 2
- net IO0: track 58.0 -> 74.6 mm
- net I2C_SDA: track 44.9 -> 60.8 mm, vias 1 -> 3
- net IO4: track 57.3 -> 70.7 mm
- net SPI_Din: track 37.2 -> 50.4 mm, vias 0 -> 2
- net SPI_SCL: track 47.1 -> 59.9 mm
- net IO2: track 66.8 -> 79.3 mm
- net SPI_Dout: track 46.6 -> 58.5 mm, vias 3 -> 5
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Other:
- board text added: "TP"
- board text added: "mlab100hw1.1"
- board text removed: "Get rid of ground under antenna"
- board text removed: "TestPlatform Rev 1.0"
