File: Electrical/TestPlatformBoard1.1/TestPlatformBoard.sch (KiCad schematic (older format))
At the start: 50 parts, among them IC1 CL520N3-G, IC2 CL520N3-G, IC3 TCR2EF33,LM(CT, IC4 ADC122S021CIMM_NOPB, IC5 DS2482-100, J1 Conn_01x04, J2 Conn_01x02_Male, J3 Conn_01x03_Male, J4 Conn_01x02_Male, J5 Conn_01x08_Male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

Commit message: v1.0
Parts:
- added MH1, MH2, MH3, MH4: MountingHole, Mounting_Holes:MountingHole_3.2mm_M3, symbol Mechanical:MountingHole
- added MH5, MH6, MH7, MH8: MountingHole, Mounting_Holes:MountingHole_3.7mm, symbol Mechanical:MountingHole
- added R14: 33k, Resistors_SMD:R_0805_HandSoldering, symbol Device:R
- J8: renamed from J?; footprint (none) -> Connectors_Samtec:SL-101-X-XX_1x01
- Q3: value DMN2041 -> DMN3404
- Q7: renamed from Q?; value Q_NMOS_GDS -> AOD4184A; footprint (none) -> TO_SOT_Packages_SMD:TO-252-2
- R3: value 330 -> 1k
- gave numbers to parts that had none: 1
Connections:
- wire segments 167 -> 171
Other:
- note removed: "3v3 Not turning on......\n"
- note removed: "ITS FUCKED, V- and A-/B- need to be switched\n"
- note removed: "Need Bigger Mosfet!\n"
- note removed: "Pair this with something beefier\n"
Changed lines of the file:
@@
 F0 "LMC6482" 50
 F1 "LMC6482.sch" 50
-F2 "A-" I L 11550 3000 50
-F3 "B-" I L 11550 3100 50
+F2 "A+" I L 11550 3000 50
+F3 "B+" I L 11550 3100 50
 F4 "V+" I L 11550 2750 50
 F5 "V-" I L 11550 3350 50
@@
 	-1   0    0    1
 $EndComp
-Wire Wire Line
-	11300 3000 11550 3000
-Wire Wire Line
-	11550 3100 10900 3100
 $Comp
 L ADC122S021CIMM_NOPB:ADC122S021CIMM_NOPB IC4
@@
 Text GLabel 12200 1850 0    50   Input ~ 0
 CTRL_3V3A
-$Comp
-L Device:Q_NMOS_GSD Q3
-U 1 1 5C05D9B5
-P 3800 5200
-F 0 "Q3" H 4005 5246 50  0000 L CNN
-F 1 "DMN2041" H 4005 5155 50  0000 L CNN
-F 2 "TO_SOT_Packages_SMD:SOT-23_Handsoldering" H 4000 5300 50  0001 C CNN
-F 3 "~" H 3800 5200 50  0001 C CNN
-	1    3800 5200
-	1    0    0    -1
-$EndComp
-$Comp
-L power:GND #PWR016
-U 1 1 5C05DB9D
-P 3900 5500
-F 0 "#PWR016" H 3900 5250 50  0001 C CNN
-F 1 "GND" H 3905 5327 50  0000 C CNN
-F 2 "" H 3900 5500 50  0001 C CNN
-F 3 "" H 3900 5500 50  0001 C CNN
-	1    3900 5500
-	1    0    0    -1
-$EndComp
-Wire Wire Line
-	3900 5500 3900 5400
+Wire Wire Line
+	3900 5550 3900 5400
 Text GLabel 4400 4500 2    50   Input ~ 0
 Heater-
-$Comp
-L Device:R R3
-U 1 1 5C062256
-P 3450 5200
-F 0 "R3" V 3243 5200 50  0000 C CNN
-F 1 "330" V 3334 5200 50  0000 C CNN
-F 2 "Resistors_SMD:R_0805_HandSoldering" V 3380 5200 50  0001 C CNN
-F 3 "~" H 3450 5200 50  0001 C CNN
-	1    3450 5200
-	0    1    1    0
-$EndComp
-Wire Wire Line
-	3250 5200 3300 5200
-Text GLabel 3250 5200 0    50   Input ~ 0
+Wire Wire Line
+	3150 5200 3200 5200
+Text GLabel 3150 5200 0    50   Input ~ 0
 CTRL_Heater
 $Comp
@@
 Text GLabel 6100 3850 0    50   Input ~ 0
 I2C_SCL
-Text Notes 5250 4850 0    200  ~ 0
-Need Bigger Mosfet!\n
-Text Notes 5450 5050 0    50   ~ 0
-Pair this with something beefier\n
-$Comp
-L Device:Q_NMOS_GDS Q?
+$Comp
+L Device:Q_NMOS_GDS Q7
 U 1 1 5C818EC7
 P 4300 4900
-F 0 "Q?" H 4506 4945 50  0000 L CNN
-F 1 "Q_NMOS_GDS" H 4506 4855 50  0000 L CNN
-F 2 "" H 4500 5000 50  0001 C CNN
+F 0 "Q7" H 4506 4945 50  0000 L CNN
+F 1 "AOD4184A" H 4506 4855 50  0000 L CNN
+F 2 "TO_SOT_Packages_SMD:TO-252-2" H 4500 5000 50  0001 C CNN
 F 3 "~" H 4300 4900 50  0001 C CNN
 	1    4300 4900
@@
 $EndComp
 $Comp
-L Device:R R?
+L Device:R R15
 U 1 1 5C819639
 P 3900 4650
-F 0 "R?" V 3693 4650 50  0000 C CNN
+F 0 "R15" V 3693 4650 50  0000 C CNN
 F 1 "1k" V 3784 4650 50  0000 C CNN
 F 2 "Resistors_SMD:R_0805_HandSoldering" V 3830 4650 50  0001 C CNN
@@
 	3900 4800 3900 4900
 $Comp
-L power:+12V #PWR?
+L power:+12V #PWR051
 U 1 1 5C822597
 P 3900 4500
-F 0 "#PWR?" H 3900 4350 50  0001 C CNN
+F 0 "#PWR051" H 3900 4350 50  0001 C CNN
 F 1 "+12V" H 3915 4673 50  0000 C CNN
 F 2 "" H 3900 4500 50  0001 C CNN
@@
 	4400 4500 4400 4700
 $Comp
-L power:GND #PWR?
+L power:GND #PWR053
 U 1 1 5C8342E3
 P 4400 5300
-F 0 "#PWR?" H 4400 5050 50  0001 C CNN
+F 0 "#PWR053" H 4400 5050 50  0001 C CNN
 F 1 "GND" H 4405 5127 50  0000 C CNN
 F 2 "" H 4400 5300 50  0001 C CNN
@@
 	4400 5300 4400 5100
 $Comp
-L Connector:Conn_01x01_Male J?
+L Connector:Conn_01x01_Male J8
 U 1 1 5C847999
 P 14000 2250
-F 0 "J?" H 13972 2181 50  0000 R CNN
+F 0 "J8" H 13972 2181 50  0000 R CNN
 F 1 "Conn_01x01_Male" H 13972 2271 50  0000 R CNN
-F 2 "" H 14000 2250 50  0001 C CNN
+F 2 "Connectors_Samtec:SL-101-X-XX_1x01" H 14000 2250 50  0001 C CNN
 F 3 "~" H 14000 2250 50  0001 C CNN
 	1    14000 2250
@@
 $EndComp
 $Comp
-L power:GNDA #PWR?
+L power:GNDA #PWR054
 U 1 1 5C847AD7
 P 13700 2350
-F 0 "#PWR?" H 13700 2100 50  0001 C CNN
+F 0 "#PWR054" H 13700 2100 50  0001 C CNN
 F 1 "GNDA" H 13705 2177 50  0000 C CNN
 F 2 "" H 13700 2350 50  0001 C CNN
@@
 Wire Wire Line
 	13700 2250 13800 2250
-Text Notes 10750 3800 0    50   ~ 0
-ITS FUCKED, V- and A-/B- need to be switched\n
-Text Notes 12650 1200 0    50   ~ 0
-3v3 Not turning on......\n
+$Comp
+L Device:Q_NMOS_GSD Q3
+U 1 1 5C377659
+P 3800 5200
+F 0 "Q3" H 4005 5246 50  0000 L CNN
+F 1 "DMN3404" H 4005 5155 50  0000 L CNN
+F 2 "TO_SOT_Packages_SMD:SOT-23_Handsoldering" H 4000 5300 50  0001 C CNN
+F 3 "~" H 3800 5200 50  0001 C CNN
+	1    3800 5200
+	1    0    0    -1
+$EndComp
+$Comp
+L Device:R R3
+U 1 1 5C377E40
+P 3350 5200
+F 0 "R3" V 3557 5200 50  0000 C CNN
+F 1 "1k" V 3466 5200 50  0000 C CNN
+F 2 "Resistors_SMD:R_0805_HandSoldering" V 3280 5200 50  0001 C CNN
+F 3 "~" H 3350 5200 50  0001 C CNN
+	1    3350 5200
+	0    -1   -1   0
+$EndComp
+$Comp
+L Device:R R14
+U 1 1 5C3786A3
+P 3550 4950
+F 0 "R14" V 3757 4950 50  0000 C CNN
+F 1 "33k" V 3666 4950 50  0000 C CNN
+F 2 "Resistors_SMD:R_0805_HandSoldering" V 3480 4950 50  0001 C CNN
+F 3 "~" H 3550 4950 50  0001 C CNN
+	1    3550 4950
+	1    0    0    -1
+$EndComp
+Wire Wire Line
+	3600 5200 3550 5200
+Connection ~ 3550 5200
+Wire Wire Line
+	3550 5200 3500 5200
+$Comp
+L power:GND #PWR052
+U 1 1 5C39D84D
+P 3900 5550
+F 0 "#PWR052" H 3900 5300 50  0001 C CNN
+F 1 "GND" H 3905 5377 50  0000 C CNN
+F 2 "" H 3900 5550 50  0001 C CNN
+F 3 "" H 3900 5550 50  0001 C CNN
+	1    3900 5550
+	1    0    0    -1
+$EndComp
+$Comp
+L power:+3.3V #PWR016
+U 1 1 5C3A806E
+P 3550 4700
+F 0 "#PWR016" H 3550 4550 50  0001 C CNN
+F 1 "+3.3V" H 3565 4873 50  0000 C CNN
+F 2 "" H 3550 4700 50  0001 C CNN
+F 3 "" H 3550 4700 50  0001 C CNN
+	1    3550 4700
+	1    0    0    -1
+$EndComp
+Wire Wire Line
+	3550 4700 3550 4800
+Wire Wire Line
+	3550 5100 3550 5200
+Wire Wire Line
+	10900 3100 11550 3100
+Wire Wire Line
+	11300 3000 11550 3000
+$Comp
+L Mechanical:MountingHole MH3
+U 1 1 5C3DEA79
+P 5350 4950
+F 0 "MH3" H 5450 4995 50  0000 L CNN
+F 1 "MountingHole" H 5450 4905 50  0000 L CNN
+F 2 "Mounting_Holes:MountingHole_3.2mm_M3" H 5350 4950 50  0001 C CNN
+F 3 "~" H 5350 4950 50  0001 C CNN
+	1    5350 4950
+	1    0    0    -1
+$EndComp
+$Comp
+L Mechanical:MountingHole MH5
+U 1 1 5C3DEC53
+P 5750 4950
+F 0 "MH5" H 5850 4995 50  0000 L CNN
+F 1 "MountingHole" H 5850 4905 50  0000 L CNN
+F 2 "Mounting_Holes:MountingHole_3.7mm" H 5750 4950 50  0001 C CNN
+F 3 "~" H 5750 4950 50  0001 C CNN
+	1    5750 4950
+	1    0    0    -1
+$EndComp
+$Comp
+L Mechanical:MountingHole MH6
+U 1 1 5C3DECD3
+P 5750 5250
+F 0 "MH6" H 5850 5295 50  0000 L CNN
+F 1 "MountingHole" H 5850 5205 50  0000 L CNN
+F 2 "Mounting_Holes:MountingHole_3.7mm" H 5750 5250 50  0001 C CNN
+F 3 "~" H 5750 5250 50  0001 C CNN
+	1    5750 5250
+	1    0    0    -1
+$EndComp
+$Comp
+L Mechanical:MountingHole MH4
+U 1 1 5C3DED5B
+P 5350 5250
+F 0 "MH4" H 5450 5295 50  0000 L CNN
+F 1 "MountingHole" H 5450 5205 50  0000 L CNN
+F 2 "Mounting_Holes:MountingHole_3.2mm_M3" H 5350 5250 50  0001 C CNN
+F 3 "~" H 5350 5250 50  0001 C CNN
+	1    5350 5250
+	1    0    0    -1
+$EndComp
+$Comp
+L Mechanical:MountingHole MH1
+U 1 1 5C3DEE68
+P 5200 4750
+F 0 "MH1" H 5300 4795 50  0000 L CNN
+F 1 "MountingHole" H 5300 4705 50  0000 L CNN
+F 2 "Mounting_Holes:MountingHole_3.2mm_M3" H 5200 4750 50  0001 C CNN
+F 3 "~" H 5200 4750 50  0001 C CNN
+	1    5200 4750
+	1    0    0    -1
+$EndComp
+$Comp
+L Mechanical:MountingHole MH7
+U 1 1 5C3DEE6F
+P 6350 4750
+F 0 "MH7" H 6450 4795 50  0000 L CNN
+F 1 "MountingHole" H 6450 4705 50  0000 L CNN
+F 2 "Mounting_Holes:MountingHole_3.7mm" H 6350 4750 50  0001 C CNN
+F 3 "~" H 6350 4750 50  0001 C CNN
+	1    6350 4750
+	1    0    0    -1
+$EndComp
+$Comp
+L Mechanical:MountingHole MH8
+U 1 1 5C3DEE76
+P 6350 5600
+F 0 "MH8" H 6450 5645 50  0000 L CNN
+F 1 "MountingHole" H 6450 5555 50  0000 L CNN
+F 2 "Mounting_Holes:MountingHole_3.7mm" H 6350 5600 50  0001 C CNN
+F 3 "~" H 6350 5600 50  0001 C CNN
+	1    6350 5600
+	1    0    0    -1
+$EndComp
+$Comp
+L Mechanical:MountingHole MH2
+U 1 1 5C3DEE7D
+P 5200 5600
+F 0 "MH2" H 5300 5645 50  0000 L CNN
+F 1 "MountingHole" H 5300 5555 50  0000 L CNN
+F 2 "Mounting_Holes:MountingHole_3.2mm_M3" H 5200 5600 50  0001 C CNN
+F 3 "~" H 5200 5600 50  0001 C CNN
+	1    5200 5600
+	1    0    0    -1
+$EndComp
 $EndSCHEMATC
