File: Electrical/mlab100_1.5/LEDBoard.sch (KiCad schematic (older format))
At the start: 5 parts, among them U4 DS18B20

Commit message: PCB 1.5 done
Parts:
- R1: footprint Resistors_SMD:R_0805_HandSoldering -> Resistors_SMD:R_1210_HandSoldering
- U4: footprint Package_TO_SOT_THT:TO-92_Inline -> TO_SOT_Packages_THT:TO-92_Molded_Narrow
Changed lines of the file:
@@
 AR Path="/5C5BF7E1/5C54DDD9" Ref="D5"  Part="1"
 AR Path="/5C5C7B67/5C54DDD9" Ref="D10"  Part="1"
-F 0 "D1" V 5936 3133 50  0000 R CNN
+F 0 "D5" V 5936 3133 50  0000 R CNN
 F 1 "470nm" V 5846 3133 50  0000 R CNN
 F 2 "LEDs:LED_D5.0mm" H 5900 3250 50  0001 C CNN
@@
 AR Path="/5C5BF7E1/5C54DFD4" Ref="D8"  Part="1"
 AR Path="/5C5C7B67/5C54DFD4" Ref="D11"  Part="1"
-F 0 "D2" V 5936 3533 50  0000 R CNN
+F 0 "D8" V 5936 3533 50  0000 R CNN
 F 1 "470nm" V 5846 3533 50  0000 R CNN
 F 2 "LEDs:LED_D5.0mm" H 5900 3650 50  0001 C CNN
@@
 AR Path="/5C5BF7E1/5C54E02C" Ref="D9"  Part="1"
 AR Path="/5C5C7B67/5C54E02C" Ref="D12"  Part="1"
-F 0 "D4" V 5936 3933 50  0000 R CNN
+F 0 "D9" V 5936 3933 50  0000 R CNN
 F 1 "470nm" V 5846 3933 50  0000 R CNN
 F 2 "LEDs:LED_D5.0mm" H 5900 4050 50  0001 C CNN
@@
 AR Path="/5C5BF7E1/5C54E391" Ref="R2"  Part="1"
 AR Path="/5C5C7B67/5C54E391" Ref="R3"  Part="1"
-F 0 "R1" H 5970 4495 50  0000 L CNN
+F 0 "R2" H 5970 4495 50  0000 L CNN
 F 1 "120" H 5970 4405 50  0000 L CNN
-F 2 "Resistors_SMD:R_0805_HandSoldering" V 5830 4450 50  0001 C CNN
+F 2 "Resistors_SMD:R_1210_HandSoldering" V 5830 4450 50  0001 C CNN
 F 3 "~" H 5900 4450 50  0001 C CNN
 	1    5900 4450
@@
 AR Path="/5C5BF7E1/5C54EB11" Ref="U5"  Part="1"
 AR Path="/5C5C7B67/5C54EB11" Ref="U6"  Part="1"
-F 0 "U4" H 6871 3695 50  0000 R CNN
+F 0 "U5" H 6871 3695 50  0000 R CNN
 F 1 "DS18B20" H 6871 3605 50  0000 R CNN
-F 2 "Package_TO_SOT_THT:TO-92_Inline" H 6100 3400 50  0001 C CNN
+F 2 "TO_SOT_Packages_THT:TO-92_Molded_Narrow" H 6100 3400 50  0001 C CNN
 F 3 "http://datasheets.maximintegrated.com/en/ds/DS18B20.pdf" H 6950 3900 50  0001 C CNN
 	1    7100 3650
