File: Electrical/mlab100_1.5/LMC6482.sch (KiCad schematic (older format))
At the start: 7 parts, among them U3 LMC6482

Commit message: PCB 1.5 done
Parts:
- C10, C9: footprint Capacitors_SMD:C_0805_HandSoldering -> Capacitors_SMD:C_0603
- R10, R11: footprint Resistors_SMD:R_1206_HandSoldering -> Resistors_SMD:R_0603
Changed lines of the file:
@@
 F 0 "R10" V 4843 2100 50  0000 C CNN
 F 1 "1M" V 4934 2100 50  0000 C CNN
-F 2 "Resistors_SMD:R_1206_HandSoldering" V 4980 2100 50  0001 C CNN
+F 2 "Resistors_SMD:R_0603" V 4980 2100 50  0001 C CNN
 F 3 "~" H 5050 2100 50  0001 C CNN
 	1    5050 2100
@@
 F 0 "C9" V 5048 1750 50  0000 C CNN
 F 1 "100pF" V 5139 1750 50  0000 C CNN
-F 2 "Capacitors_SMD:C_0805_HandSoldering" H 5338 1600 50  0001 C CNN
+F 2 "Capacitors_SMD:C_0603" H 5338 1600 50  0001 C CNN
 F 3 "~" H 5300 1750 50  0001 C CNN
 	1    5300 1750
@@
 F 0 "R11" V 4843 3450 50  0000 C CNN
 F 1 "1M" V 4934 3450 50  0000 C CNN
-F 2 "Resistors_SMD:R_1206_HandSoldering" V 4980 3450 50  0001 C CNN
+F 2 "Resistors_SMD:R_0603" V 4980 3450 50  0001 C CNN
 F 3 "~" H 5050 3450 50  0001 C CNN
 	1    5050 3450
@@
 F 0 "C10" V 5048 3100 50  0000 C CNN
 F 1 "100pF" V 5139 3100 50  0000 C CNN
-F 2 "Capacitors_SMD:C_0805_HandSoldering" H 5338 2950 50  0001 C CNN
+F 2 "Capacitors_SMD:C_0603" H 5338 2950 50  0001 C CNN
 F 3 "~" H 5300 3100 50  0001 C CNN
 	1    5300 3100
