File: Electrical/mlab100_1.5/mlab100_1.5.kicad_pcb (KiCad board)
At the start: 2 copper layers, 88.9 x 76.2 mm, 79 parts, among them IC1 ZXGD3006E6QTA, IC2 ZXGD3006E6QTA, IC3 TCR2EF33,LM(CT, IC4 ADC122S021CIMM_NOPB, J1 Conn_01x04, J10 Conn_01x06_Male, J11 Conn_01x02_Male, J12 Conn_01x02_Male, J13 Conn_01x02_Male, J14 Conn_01x06_Male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

Commit message: PCB 1.5 done
Parts:
- removed C6, C7: 1uF, Capacitors_SMD:C_0805_HandSoldering
- removed C8: 0.1uF, Capacitors_SMD:C_0805_HandSoldering
- removed J17: Conn_01x01_Male, Pin_Headers:Pin_Header_Straight_1x01_Pitch2.54mm
- added MH10: MountingHole, Mounting_Holes:MountingHole_3.7mm_Pad, F.Cu at (143.5, 25.5)
- added MH8: MountingHole, Mounting_Holes:MountingHole_3.7mm_Pad, F.Cu at (143.5, 53.2)
- added MH9: MountingHole, Mounting_Holes:MountingHole_3.7mm_Pad, F.Cu at (119.5, 39.4)
- added U4: DS18B20, TO_SOT_Packages_THT:TO-92_Molded_Narrow, F.Cu at (2.96, 94.6)
- added U5: DS18B20, TO_SOT_Packages_THT:TO-92_Molded_Narrow, F.Cu at (2.96, 87.8)
- added U6: DS18B20, TO_SOT_Packages_THT:TO-92_Molded_Narrow, F.Cu at (2.96, 81.1)
- C1, C10, C2, C5, C9: footprint Capacitors_SMD:C_0805_HandSoldering -> Capacitors_SMD:C_0603; moved to B.Cu
- IC1, IC2, IC3, IC4, J10, J3, J8, J9, Q1, Q3, U3: moved to B.Cu
- JP1, R14, R15, R16: footprint Resistors_SMD:R_0805_HandSoldering -> Resistors_SMD:R_0603; moved to B.Cu
- R1, R2, R3: footprint Resistors_SMD:R_0805_HandSoldering -> Resistors_SMD:R_1210_HandSoldering
- R10, R11: footprint Resistors_SMD:R_1206_HandSoldering -> Resistors_SMD:R_0603; moved to B.Cu
- R12, R13: footprint Resistors_SMD:R_0805_HandSoldering -> Resistors_SMD:R_0603
- moved D1 251.0 mm to (7.94, 93.3), turned to 0 degrees
- moved D5 249.5 mm to (7.94, 86.6), turned to 0 degrees
- moved D10 244.7 mm to (7.94, 79.8)
- moved D2 235.5 mm to (14.4, 93.3)
- moved D8 233.5 mm to (14.4, 86.6)
- moved D11 231.7 mm to (14.4, 79.8)
- moved D4 221.9 mm to (20.9, 93.3), turned to 0 degrees
- moved D9 220.7 mm to (20.9, 86.6)
- moved D12 218.7 mm to (20.9, 79.8)
- moved R1 192.2 mm to (43.0, 93.3)
- moved R2 191.4 mm to (43.0, 86.6)
- moved J15 187.4 mm to (54.5, 85.3)
- moved R3 186.9 mm to (43.0, 79.8), turned to 0 degrees
- moved J14 184.3 mm to (54.5, 92.0)
- moved J16 177.1 mm to (54.5, 78.6)
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Connections:
- net /AnalogConnPCB/SPI_CD_ADC renamed /AnalogConnPCB/SPI_CS_ADC
- J14 pad 3: (no net) -> /LEDBoard1/Temp1w
- J14 pad 5: (no net) -> /LEDBoard1/3V3
- J15 pad 3: (no net) -> /LEDBoard2/Temp1w
- J15 pad 5: (no net) -> /LEDBoard2/3V3
- J16 pad 3: (no net) -> /LEDBoard3/Temp1w
- J16 pad 5: (no net) -> /LEDBoard3/3V3
- J2 pad 1: +12V -> CTRL_470nm
- J2 pad 10: CTRL_Heater -> SPI_CS_ADC
- J2 pad 11: CTRL_470nm -> CTRL_Heater
- J2 pad 12: TEMP1W -> +5V
- J2 pad 2: +5V -> +12V
- J2 pad 3: +3V3 -> TEMP1W
- J2 pad 4: GND -> +3V3
- J2 pad 5: CTRL_3V3A -> SPI_SCL
- J2 pad 6: SPI_SCL -> CTRL_3V3A
- J2 pad 9: SPI_CS_ADC -> GND
- J3 pad 10: /AnalogConnPCB/HeaterCtrl -> GND_O
- J3 pad 11: /AnalogConnPCB/470nmCtrl -> /AnalogConnPCB/5V
- J3 pad 12: Temp1wDaisy -> /AnalogConnPCB/HeaterCtrl
- J3 pad 2: /AnalogConnPCB/5V -> /AnalogConnPCB/470nmCtrl
- J3 pad 4: GND_O -> Temp1wDaisy
- J3 pad 7: /AnalogConnPCB/SPI_MISO -> /AnalogConnPCB/SPI_MOSI
- J3 pad 8: /AnalogConnPCB/SPI_MOSI -> /AnalogConnPCB/SPI_MISO
Routing:
- net 12V_O: track 0.00 -> 153.6 mm, vias 0 -> 7
- net SPI_MISO: track 0.00 -> 110.2 mm, vias 0 -> 3
- net SPI_MOSI: track 0.00 -> 95.5 mm, vias 0 -> 3
- net LED470nm: track 0.00 -> 94.7 mm, vias 0 -> 3
- net SPI_CS_ADC: track 7.50 -> 101.0 mm, vias 0 -> 3
- net Heater-: track 0.00 -> 88.4 mm
- net LED_R: track 2.47 -> 84.2 mm
- net LED_Y: track 2.45 -> 79.9 mm
- net Temp1wDaisy: track 0.00 -> 74.8 mm, vias 0 -> 3
- net LED_G: track 2.52 -> 75.6 mm
- net 3V3_O: track 0.00 -> 72.1 mm, vias 0 -> 2
- net CTRL_Heater: track 0.04 -> 69.2 mm, vias 0 -> 1
- net +12V: track 45.5 -> 111.2 mm
- net CTRL_470nm: track 0.00 -> 63.3 mm, vias 0 -> 2
- net /LEDBoard3/Temp1w: track 0.00 -> 55.8 mm
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- added copper zone on B.Cu, net /LEDBoard1/GND
- added copper zone on F.Cu, net /LEDBoard1/GND
- added copper zone on B.Cu, net /LEDBoard2/GND
- added copper zone on F.Cu, net /LEDBoard2/GND
- added copper zone on B.Cu, net /LEDBoard3/GND
- added copper zone on F.Cu, net /LEDBoard3/GND
- added copper zone on B.Cu, net GNDA
- added copper zone on F.Cu, net GNDA
- added copper zone on B.Cu, net GND_O
- added copper zone on F.Cu, net GND_O
Other:
- board size 88.9 x 76.2 mm -> 155.5 x 96.2 mm
- board text added: "12V 5V0 3V3 GND"
- board text added: "GPIO"
- board text added: "I2C"
- board text added: "MBlab100 V1.5"
- board text added: "MicroBiota Labs Inc"
- board text added: "SPI"
- board text removed: "MicroBiota Lab Inc"
- board text removed: "mlab100hw1.1"
